File: pcb/minivol_led_encoder/minivol_led_encoder.kicad_pcb (KiCad board)
At the start: 2 copper layers, 66 x 57.2 mm, 26 parts, among them J1 Encoder and SPI input, J3 Encoder output, U1 74HC595

Commit message: flat cam CNC jobs
Routing:
- net Net-(D3-Pad2): track 26.5 -> 27.4 mm
- net Net-(D1-Pad2): track 33.0 -> 33.8 mm
Changed lines of the file:
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@@
     (thickness 1.6)
     (drawings 9)
-    (tracks 118)
+    (tracks 116)
     (zones 0)
     (modules 26)
@@
     (pad_drill 3.2)
     (pad_to_mask_clearance 0.2)
-    (aux_axis_origin 0 0)
+    (aux_axis_origin 116 126)
+    (grid_origin 116 126)
     (visible_elements FFFFFF7F)
     (pcbplotparams
@@
       (viasonmask false)
       (mode 1)
-      (useauxorigin false)
+      (useauxorigin true)
       (hpglpennumber 1)
       (hpglpenspeed 20)
@@
       (effects (font (size 1 1) (thickness 0.15)))
     )
-    (pad 1 np_thru_hole circle (at 0 0) (size 3.2 3.2) (drill 3.2) (layers *.Cu *.Mask))
+    (pad "" np_thru_hole circle (at 0 0) (size 3.2 3.2) (drill 3.2) (layers *.Cu *.Mask))
   )
   (module Mounting_Holes:MountingHole_3.2mm_M3 (layer F.Cu)
@@
   (segment (start 148.59 99.06) (end 147.790001 99.859999) (width 0.5) (layer B.Cu) (net 5) (status 10))
   (segment (start 147.790001 99.859999) (end 147.790001 101.267219) (width 0.5) (layer B.Cu) (net 5))
-  (segment (start 162.029999 100.860001) (end 173.350001 89.539999) (width 0.5) (layer B.Cu) (net 6))
-  (segment (start 173.350001 89.539999) (end 178.442791 89.539999) (width 0.5) (layer B.Cu) (net 6))
-  (segment (start 178.442791 89.539999) (end 179.07 90.167208) (width 0.5) (layer B.Cu) (net 6))
-  (segment (start 179.07 90.167208) (end 179.07 91.44) (width 0.5) (layer B.Cu) (net 6) (status 20))
-  (segment (start 153.67 99.06) (end 153.67 100.19137) (width 0.5) (layer B.Cu) (net 6) (status 10))
-  (segment (start 153.67 100.19137) (end 154.338631 100.860001) (width 0.5) (layer B.Cu) (net 6))
-  (segment (start 154.338631 100.860001) (end 162.029999 100.860001) (width 0.5) (layer B.Cu) (net 6))
+  (segment (start 179.07 91.44) (end 179.07 96.644002) (width 0.5) (layer B.Cu) (net 6))
+  (segment (start 179.07 96.644002) (end 174.854001 100.860001) (width 0.5) (layer B.Cu) (net 6))
+  (segment (start 174.854001 100.860001) (end 154.338631 100.860001) (width 0.5) (layer B.Cu) (net 6))
+  (segment (start 154.338631 100.860001) (end 153.67 100.19137) (width 0.5) (layer B.Cu) (net 6))
+  (segment (start 153.67 100.19137) (end 153.67 99.06) (width 0.5) (layer B.Cu) (net 6))
   (segment (start 176.53 91.44) (end 176.53 96.52) (width 0.5) (layer B.Cu) (net 7) (status 30))
   (segment (start 173.99 82.55) (end 173.99 81.277208) (width 0.5) (layer B.Cu) (net 8) (status 10))
@@
   (segment (start 171.45 82.55) (end 171.45 87.63) (width 0.5) (layer B.Cu) (net 9) (status 30))
   (segment (start 163.83 81.28) (end 163.83 76.2) (width 0.5) (layer B.Cu) (net 10) (status 30))
-  (segment (start 153.67 91.44) (end 153.67 90.30863) (width 0.5) (layer B.Cu) (net 11) (status 10))
-  (segment (start 153.67 90.30863) (end 161.879999 82.098631) (width 0.5) (layer B.Cu) (net 11))
-  (segment (start 162.089999 74.249999) (end 165.692791 74.249999) (width 0.5) (layer B.Cu) (net 11))
-  (segment (start 161.879999 82.098631) (end 161.879999 74.459999) (width 0.5) (layer B.Cu) (net 11))
-  (segment (start 161.879999 74.459999) (end 162.089999 74.249999) (width 0.5) (layer B.Cu) (net 11))
-  (segment (start 166.37 74.927208) (end 166.37 76.2) (width 0.5) (layer B.Cu) (net 11) (status 30))
-  (segment (start 165.692791 74.249999) (end 166.37 74.927208) (width 0.5) (layer B.Cu) (net 11) (status 20))
+  (segment (start 161.085 74.709998) (end 161.085 82.89363) (width 0.5) (layer B.Cu) (net 11))
+  (segment (start 161.085 82.89363) (end 153.67 90.30863) (width 0.5) (layer B.Cu) (net 11))
+  (segment (start 153.67 90.30863) (end 153.67 91.44) (width 0.5) (layer B.Cu) (net 11))
+  (segment (start 165.372792 73.295) (end 162.499998 73.295) (width 0.5) (layer B.Cu) (net 11))
+  (segment (start 162.499998 73.295) (end 161.085 74.709998) (width 0.5) (layer B.Cu) (net 11))
+  (segment (start 166.37 75.565) (end 166.37 74.292208) (width 0.5) (layer B.Cu) (net 11))
+  (segment (start 166.37 74.292208) (end 165.372792 73.295) (width 0.5) (layer B.Cu) (net 11))
   (segment (start 154.305 77.47) (end 154.305 72.39) (width 0.5) (layer B.Cu) (net 12) (status 30))
   (segment (start 151.13 91.44) (end 151.13 83.309002) (width 0.5) (layer B.Cu) (net 13) (status 10))
